Commit message: 重力标定改用双向逼近消除静摩擦
静止时力矩平衡是 tau_applied + G + tau_f = 0，而摩擦在 [-tau_s, +tau_s] 内取值
不定——静力平衡对它欠定。静摩擦总是反抗最后一次运动的方向，所以单向逼近时它在
所有样本里同号，被回归当成系统项，一部分进 torque_bias、一部分抬高质量。实测
tau_s 为 0.05~0.77 N.m，占重力矩的 5~50%，而改进前左臂的标定残差中位 0.081 N.m
恰好落在同一量级：残差主要是摩擦，不是模型误差。

改法是每个姿态采两次，先退开再从两侧各回到目标一次，两个 StaticSample 取平均：

    tau_up = -G + f,  tau_down = -G - f  =>  (tau_up + tau_down)/2 = -G

摩擦项恒等消去，与 f 多大无关。拟合代码一行未改。

- 必须先退开再回来：直接走到目标点的话方向取决于手臂原先在哪，两次可能同向
- 退让幅度 approach_offset_rad 默认 0.12 rad，必须大于死区 2*tau_s/kp（实测最大
  0.107），小于死区则关节没挪到另一侧、两次停在同一点，平均下来等于没做
- 差值的一半就是该点的摩擦力矩，记入 StaticSample.friction 并随迭代落盘，
  每侧标定结束时打印。它不进回归，是白拿的副产物
- 代价是标定时间约 4 倍（每姿态 4 次移动 + 2 个静态窗口）

同时把 URDF 身份校验从整份文件的 sha256 改成只覆盖运动学与惯量的模型摘要：
关节的连接关系/origin/axis/limit 与连杆的 inertial，忽略 visual/collision/material。
改一次渲染颜色就被判成换了机器人、标定节点拒绝启动，这次实机撞上了。旧格式的参数
文件内容未变时就地升级；已经改过渲染的用 rebind_urdf:=true 一次性接受，采样点、
model_scope 与 links 全部保留（实测 11 targets / 108 links 无损）。

实测（11 个姿态，双向 vs 单向）：
  rank/nullity   10/4      -> 11/3
  rmse_after     0.53~0.60 -> 0.11~0.14
  最大尺度偏离   2.21      -> 1.25

零空间漂移随之不再是问题：它的根因就是摩擦被塞进不可辨识方向。README 里那段
"对称化平均"的建议同时删除——它的前提是两臂硬件相同，而右臂已经换过。

含本次重新标定的 parameters.json / calibrated.urdf / gravity_table.yaml /
ft_calibration.yaml。数学推导见新增的 CALIBRATION.md。

补：同一批数据显示摩擦正比于关节载荷，tau_f ~= mu*|tau_g| + tau0，mu 落在
0.13~0.22，各关节与两侧高度一致（相关系数左臂 0.71~0.96）。这是后续做摩擦补偿的
前提——同一关节的摩擦跨位姿能差 11 倍，按中位数做常数补偿会在轻载位姿过补 10 倍、
等于接了负阻尼。早先把这 30% 的跨位姿离散当成测量噪声是误读。

File: src/arm_gravity_compensation/config/calibrated.urdf (robot description, URDF)
Before this commit: robot g1_with_dual_gloria_m, 108 links, 107 joints
Links:
- link left_eccentric: mass 0.029687330116124018 -> 0.027974822850963324
- link left_elbow_link: mass 0.80908115271697001 -> 0.61526775453980498
- link left_gripper_base: mass 0.44722251443870648 -> 0.42142457969267316
- link left_kwr57b_link: mass 0.34749566819009242 -> 0.32745045516286253
- link left_left_connecting_rod: mass 0.008590079552441076 -> 0.0080945626573776866
- link left_left_slider: mass 0.087085448352924824 -> 0.082061942958171888
- link left_right_connecting_rod: mass 0.008590079552441076 -> 0.0080945626573776866
- link left_right_slider: mass 0.087085448352924824 -> 0.082061942958171888
- link left_shoulder_pitch_link: mass 0.64885876347088633 -> 0.57569378657234782
- link left_shoulder_roll_link: mass 0.84214224073079758 -> 0.60930923021085548
- link left_shoulder_yaw_link: mass 1.4666459619647374 -> 0.89388254204489592
- link left_wrist_pitch_link: mass 0.46737746040628725 -> 0.83710792661614175
- link left_wrist_roll_link: mass 0.082447764775937349 -> 0.08533403118227012
- link left_wrist_yaw_link: mass 0.11303829598388193 -> 0.10651770614449303
- link right_eccentric: mass 0.029687330116124018 -> 0.026680055699111641
- link right_elbow_link: mass 0.80908115271697001 -> 0.61140767133954499
- link right_gripper_base: mass 0.44722251443870648 -> 0.4019196589403265
- link right_kwr57b_link: mass 0.34749566819009242 -> 0.31229496712054389
- link right_left_connecting_rod: mass 0.008590079552441076 -> 0.0077199195758749549
- link right_left_slider: mass 0.087085448352924824 -> 0.078263845335698162
- link right_right_connecting_rod: mass 0.008590079552441076 -> 0.0077199195758749549
- link right_right_slider: mass 0.087085448352924824 -> 0.078263845335698162
- link right_shoulder_pitch_link: mass 0.64885876347088633 -> 0.6668104711265247
- link right_shoulder_roll_link: mass 0.84214224073079758 -> 0.65880103167832693
- link right_shoulder_yaw_link: mass 1.4666459619647374 -> 0.94745609323914526
- link right_wrist_pitch_link: mass 0.46737746040628725 -> 0.86725681746081107
- link right_wrist_roll_link: mass 0.082447764775937349 -> 0.082703031117021292
- link right_wrist_yaw_link: mass 0.11303829598388193 -> 0.10158771506854486
